Commit message: Add moon_surface11 terrain model

File: ros2_ws/src/mybot_description/urdf/lunabot_sensors.urdf (robot description, URDF)
Before this commit: robot lunabot, 12 links, 11 joints
Joints:
- joint base_footprint_joint: origin xyz=0 0 0.325 rpy=0 0 -1.5708 -> xyz=0 0 0.325 rpy=0 0 0
- joint camera_mount_joint: origin xyz=0 0 0.175 rpy=0 0 -1.5708 -> xyz=0 0 0.175 rpy=0 0 0
- joint depth_camera_joint: origin xyz=0.46 0 -0.14 rpy=0 0.7 0 -> xyz=0.575 0 0 rpy=0 0.35 0; parent camera_mount_link -> base_link
- joint rgb_camera_joint: origin xyz=0.275 0 0 rpy=0 0 -1.5708 -> xyz=0.275 0 0 rpy=0 0 0
